File: byteworker.kicad_pcb (KiCad board)
At the start: 2 copper layers, 34 x 34 mm, 65 parts, among them IC2 TJA1043, IC3 UA78M05IDCY, J2 AVRSPI-61.27, Q1 BSS138, Q2 BSS138, Q3 BSS138, Q4 AP2321GN-HF-3TR, Q5 BSS138, X1 16 MHz, X2 SUBD-M_H9

Commit message: some problems with too long timestamps fixed
Other:
- board text added: "K1"
- board text added: "K1: KL30 ON/OFF K2: PC Switch"
- board text added: "K2"
